File: BMP581_PCB/MainBoard/MainBoard.kicad_sch (KiCad schematic)
At the start: 8 parts, among them U1 Teensy4.1

Commit message: update strips
Parts:
- removed master_connector_input7: std_master_input, symbol BMP581_symbol:std_master_input
- added master_connector_input10, master_connector_input11, master_connector_input12, master_connector_input13, master_connector_input8, master_connector_input9: std_master_input, BMP581:Master_pins_bottom, symbol BMP581_symbol:std_master_input
- U1: footprint (none) -> BMP581:Teensy41
- master_connector_input1, master_connector_input2, master_connector_input3, master_connector_input4, master_connector_input5, master_connector_input6: footprint (none) -> BMP581:Master_pins_top
Connections:
- net at U1.46 (3V3), master_connector_input1.1 (VDDIO), master_connector_input2.1 (VDDIO)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: now also master_connector_input10.1 (VDDIO), master_connector_input11.1 (VDDIO), master_connector_input12.1 (VDDIO), master_connector_input13.1 (VDDIO), master_connector_input8.1 (VDDIO), master_connector_input9.1 (VDDIO)
- net at U1.47 (GND), master_connector_input1.2 (GND), master_connector_input2.2 (GND)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: now also master_connector_input10.2 (GND), master_connector_input11.2 (GND), master_connector_input12.2 (GND), master_connector_input13.2 (GND), master_connector_input8.2 (GND), master_connector_input9.2 (GND)
- net at master_connector_input1.3 (VDD), master_connector_input2.3 (VDD), master_connector_input3.3 (VDD)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: now also U1.15 (3V3), master_connector_input10.3 (VDD), master_connector_input11.3 (VDD), master_connector_input12.3 (VDD), master_connector_input13.3 (VDD), master_connector_input8.3 (VDD), master_connector_input9.3 (VDD); no longer U1.35 (13_SCK_LED), U1.40 (18_A4_SDA), master_connector_input3.10 (CS2)
- net at master_connector_input1.4 (SCK), master_connector_input2.4 (SCK), master_connector_input3.11 (CS2)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: now also U1.35 (13_SCK_LED), U1.40 (18_A4_SDA), master_connector_input10.11 (CS2); no longer U1.14 (12_MISO_MQSL), U1.41 (19_A5_SCL)
- net at master_connector_input1.5 (MISO), master_connector_input2.5 (MISO), master_connector_input3.12 (CS3)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: now also U1.14 (12_MISO_MQSL), U1.41 (19_A5_SCL), master_connector_input10.12 (CS3); no longer U1.13 (11_MOSI_CTX1), U1.42 (20_A6_TX5_LRCLK1)
- net at master_connector_input1.6 (MOSI), master_connector_input2.6 (MOSI), master_connector_input3.6 (MOSI)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: now also U1.13 (11_MOSI_CTX1), U1.42 (20_A6_TX5_LRCLK1), master_connector_input3.13 (CS4), master_connector_input10.13 (CS4); no longer U1.19 (27_A13_SCK1)
- net at master_connector_input5.10 (CS1): now also U1.8 (6_OUT1D), master_connector_input12.10 (CS1); no longer U1.9 (7_RX2_OUT1A)
- net at master_connector_input5.11 (CS2): now also U1.9 (7_RX2_OUT1A), master_connector_input12.11 (CS2); no longer U1.10 (8_TX2_IN1)
- net at master_connector_input5.12 (CS3): now also U1.10 (8_TX2_IN1), master_connector_input12.12 (CS3); no longer U1.11 (9_OUT1C)
- net at master_connector_input5.13 (CS4): now also U1.11 (9_OUT1C), master_connector_input12.13 (CS4); no longer U1.12 (10_CS_MQSR)
- net at master_connector_input5.14 (CS5): now also U1.12 (10_CS_MQSR), master_connector_input12.14 (CS5); no longer U1.16 (24_A10_TX6_SCL2)
- net at master_connector_input5.9 (MOSI1): no longer U1.8 (6_OUT1D)
- net at master_connector_input6.10 (CS1): now also U1.17 (25_A11_RX6_SDA2), master_connector_input13.10 (CS1); no longer U1.20 (28_RX7)
- net at master_connector_input6.11 (CS2): now also U1.20 (28_RX7), master_connector_input13.11 (CS2); no longer U1.21 (29_TX7)
- net at master_connector_input6.12 (CS3): now also U1.21 (29_TX7), master_connector_input13.12 (CS3); no longer U1.22 (30_CRX3)
- net at master_connector_input6.13 (CS4): now also U1.22 (30_CRX3), master_connector_input13.13 (CS4); no longer U1.23 (31_CTX3)
- net at master_connector_input6.14 (CS5): now also U1.23 (31_CTX3), master_connector_input13.14 (CS5); no longer U1.24 (32_OUT1B)
- net at master_connector_input6.9 (MOSI1): no longer U1.17 (25_A11_RX6_SDA2)
- net at master_connector_input4.10 (CS1): now also U1.45 (23_A9_CRX1_MCLK1), master_connector_input11.10 (CS1); no longer U1.2 (0_RX1_CRX2_CS1)
- net at master_connector_input4.11 (CS2): now also U1.2 (0_RX1_CRX2_CS1), master_connector_input11.11 (CS2); no longer U1.4 (2_OUT2)
- net at master_connector_input4.12 (CS3): now also U1.4 (2_OUT2), master_connector_input11.12 (CS3); no longer U1.5 (3_LRCLK2)
- net at master_connector_input4.13 (CS4): now also U1.5 (3_LRCLK2), master_connector_input11.13 (CS4); no longer U1.6 (4_BCLK2)
- net at master_connector_input4.14 (CS5): now also U1.6 (4_BCLK2), master_connector_input11.14 (CS5); no longer U1.7 (5_IN2)
- net at master_connector_input4.9 (MOSI1): no longer U1.45 (23_A9_CRX1_MCLK1)
- net at U1.25 (33_MCLK2): now also master_connector_input1.10 (CS1), master_connector_input8.10 (CS1); no longer master_connector_input1.9 (CS1)
- net at U1.26 (34_RX8): now also master_connector_input1.11 (CS2), master_connector_input8.11 (CS2); no longer master_connector_input1.10 (CS2)
- net at U1.27 (35_TX8): now also master_connector_input1.12 (CS3), master_connector_input8.12 (CS3); no longer master_connector_input1.11 (CS3)
- net at U1.28 (36_CS): now also master_connector_input1.13 (CS4), master_connector_input8.13 (CS4); no longer master_connector_input1.12 (CS4)
- net at U1.29 (37_CS): now also master_connector_input1.14 (CS5), master_connector_input8.14 (CS5); no longer master_connector_input1.13 (CS5)
- net at U1.30 (38_CS1_IN1): now also master_connector_input1.15 (CS6), master_connector_input8.15 (CS6); no longer master_connector_input1.14 (CS6)
- net at U1.31 (39_MISO1_OUT1A): now also master_connector_input2.10 (CS1), master_connector_input9.10 (CS1); no longer master_connector_input2.9 (CS1)
- net at U1.32 (40_A16): now also master_connector_input2.11 (CS2), master_connector_input9.11 (CS2); no longer master_connector_input2.10 (CS2)
- net at U1.33 (41_A17): now also master_connector_input2.12 (CS3), master_connector_input9.12 (CS3); no longer master_connector_input2.11 (CS3)
- net at U1.36 (14_A0_TX3_SPDIF_OUT): now also master_connector_input2.13 (CS4), master_connector_input9.13 (CS4); no longer master_connector_input2.12 (CS4)
- net at U1.37 (15_A1_RX3_SPDIF_IN): now also master_connector_input2.14 (CS5), master_connector_input9.14 (CS5); no longer master_connector_input2.13 (CS5)
- net at U1.38 (16_A2_RX4_SCL1): now also master_connector_input2.15 (CS6), master_connector_input9.15 (CS6); no longer master_connector_input2.14 (CS6)
- net at U1.39 (17_A3_TX4_SDA1): now also master_connector_input3.10 (CS1), master_connector_input10.10 (CS1); no longer master_connector_input3.9 (CS1)
- net at U1.43 (21_A7_RX5_BCLK1): now also master_connector_input3.14 (CS5), master_connector_input10.14 (CS5); no longer master_connector_input3.13 (CS5)
- net at U1.44 (22_A8_CTX1): now also master_connector_input3.15 (CS6), master_connector_input10.15 (CS6); no longer master_connector_input3.14 (CS6)
- new net: U1.19 (27_A13_SCK1), master_connector_input10.7 (SCK1), master_connector_input11.7 (SCK1), master_connector_input12.7 (SCK1), master_connector_input13.7 (SCK1), master_connector_input8.7 (SCK1), master_connector_input9.7 (SCK1)
- new net: U1.3 (1_TX1_CTX2_MISO1), master_connector_input10.8 (MISO1), master_connector_input11.8 (MISO1), master_connector_input12.8 (MISO1), master_connector_input13.8 (MISO1), master_connector_input8.8 (MISO1), master_connector_input9.8 (MISO1)
- new net: U1.18 (26_A12_MOSI1), master_connector_input10.9 (MOSI1), master_connector_input11.9 (MOSI1), master_connector_input12.9 (MOSI1), master_connector_input13.9 (MOSI1), master_connector_input8.9 (MOSI1), master_connector_input9.9 (MOSI1)
- new net: U1.7 (5_IN2), master_connector_input11.15 (CS6), master_connector_input4.15 (CS6)
- new net: U1.24 (32_OUT1B), master_connector_input13.15 (CS6), master_connector_input6.15 (CS6)
- new net: U1.16 (24_A10_TX6_SCL2), master_connector_input12.15 (CS6), master_connector_input5.15 (CS6)
- now unconnected: master_connector_input1.7 (MISO1), master_connector_input1.8 (MOSI1), master_connector_input2.7 (MISO1), master_connector_input2.8 (MOSI1), master_connector_input3.7 (MISO1), master_connector_input3.8 (MOSI1), master_connector_input4.7 (MISO1), master_connector_input4.8 (MOSI1), master_connector_input5.7 (MISO1), master_connector_input5.8 (MOSI1), master_connector_input6.7 (MISO1), master_connector_input6.8 (MOSI1)
Other:
- moved on the sheet: U1
