File: BMP581_PCB/SensorStrip_Bottom/SensorStrip_Bottom.kicad_pcb (KiCad board)
At the start: 2 copper layers, 16 parts

Commit message: update strips
Parts:
- removed the R1 at (149.5, 106.9)
- BottomStrip1: renamed from master_connector_input1; footprint Connector_PinHeader_1.27mm:PinHeader_2x14_P1.27mm_Horizontal -> BMP581:Strip_pins_bottom
- C1, C2: value 600nF -> 470nF; footprint Capacitor_SMD:C_1210_3225Metric_Pad1.33x2.70mm_HandSolder -> Capacitor_SMD:C_0603_1608Metric
- R1: renamed from R7; value 10000 -> 10k; footprint Resistor_SMD:R_01005_0402Metric_Pad0.57x0.30mm_HandSolder -> Resistor_SMD:R_0402_1005Metric
- R2: renamed from R6; value 10000 -> 10k; footprint Resistor_SMD:R_01005_0402Metric_Pad0.57x0.30mm_HandSolder -> Resistor_SMD:R_0402_1005Metric
- R3: renamed from R5; value 10000 -> 10k; footprint Resistor_SMD:R_01005_0402Metric_Pad0.57x0.30mm_HandSolder -> Resistor_SMD:R_0402_1005Metric
- R4: value 10000 -> 10k; footprint Resistor_SMD:R_01005_0402Metric_Pad0.57x0.30mm_HandSolder -> Resistor_SMD:R_0402_1005Metric
- R5: renamed from R3; value 10000 -> 10k; footprint Resistor_SMD:R_01005_0402Metric_Pad0.57x0.30mm_HandSolder -> Resistor_SMD:R_0402_1005Metric
- R6: renamed from R2; value 10000 -> 10k; footprint Resistor_SMD:R_01005_0402Metric_Pad0.57x0.30mm_HandSolder -> Resistor_SMD:R_0402_1005Metric
- moved BottomStrip1 196.5 mm to (285.1, 59.2), turned to 30.97 degrees
- moved R1 142.5 mm to (15.8, 67.5), turned to 180 degrees
- moved R2 116.1 mm to (43.4, 68.0), turned to -90 degrees
- moved R6 109.8 mm to (251.5, 68.0), turned to -90 degrees
- moved C2 102.7 mm to (261.3, 69.5), turned to -90 degrees
- moved C1 95.2 mm to (265.5, 68.5), turned to 90 degrees
- moved U1 92.7 mm to (15.5, 60.0)
- moved U2 89.0 mm to (45.2, 60.0)
- moved R3 88.8 mm to (73.2, 68.0), turned to -90 degrees
- moved R5 83.5 mm to (221.6, 68.0), turned to -90 degrees
- moved U3 79.7 mm to (74.8, 60.0)
- moved R4 60.8 mm to (191.6, 68.0), turned to -90 degrees
- moved U6 60.8 mm to (252.5, 60.0)
- moved U4 39.7 mm to (193.3, 60.0)
- moved U5 36.6 mm to (222.9, 60.0)
Connections:
- BottomStrip1 pad 1: Net-(master_connector_input1-3.3V) -> Net-(BottomStrip1-VDDIO)
- BottomStrip1 pad 10: Net-(U5-CSB) -> Net-(BottomStrip1-CS1)
- BottomStrip1 pad 11: Net-(U4-CSB) -> Net-(BottomStrip1-CS2)
- BottomStrip1 pad 12: Net-(U3-CSB) -> Net-(BottomStrip1-CS3)
- BottomStrip1 pad 13: Net-(U2-CSB) -> Net-(BottomStrip1-CS4)
- BottomStrip1 pad 14: Net-(U1-CSB) -> Net-(BottomStrip1-CS5)
- BottomStrip1 pad 15: (no net) -> Net-(BottomStrip1-CS6)
- BottomStrip1 pad 2: Net-(master_connector_input1-GND) -> GND
- BottomStrip1 pad 3: unconnected-(master_connector_input1-SCK-Pad3) -> Net-(BottomStrip1-VDD)
- BottomStrip1 pad 6: Net-(U1-SCK) -> unconnected-(BottomStrip1-MOSI-Pad6)
- BottomStrip1 pad 7: Net-(U1-SDO) -> Net-(BottomStrip1-SCK1)
- BottomStrip1 pad 8: Net-(U1-SDI) -> Net-(BottomStrip1-MISO1)
- BottomStrip1 pad 9: Net-(U6-CSB) -> Net-(BottomStrip1-MOSI1)
- C1 pad 2: Net-(U1-VDD) -> Net-(BottomStrip1-VDD)
- C2 pad 2: Net-(U1-VDDIO) -> Net-(BottomStrip1-VDDIO)
- R1 pad 1: Net-(U1-VDD) -> Net-(BottomStrip1-VDD)
- R1 pad 2: Net-(U1-CSB) -> Net-(BottomStrip1-CS6)
- R2 pad 1: Net-(U1-VDD) -> Net-(BottomStrip1-VDD)
- R2 pad 2: Net-(U2-CSB) -> Net-(BottomStrip1-CS5)
- R3 pad 1: Net-(U1-VDD) -> Net-(BottomStrip1-VDD)
- R3 pad 2: Net-(U3-CSB) -> Net-(BottomStrip1-CS4)
- R4 pad 1: Net-(U1-VDD) -> Net-(BottomStrip1-VDD)
- R4 pad 2: Net-(U4-CSB) -> Net-(BottomStrip1-CS3)
- R5 pad 1: Net-(U1-VDD) -> Net-(BottomStrip1-VDD)
- R5 pad 2: Net-(U5-CSB) -> Net-(BottomStrip1-CS2)
- R6 pad 1: Net-(U1-VDD) -> Net-(BottomStrip1-VDD)
- R6 pad 2: Net-(U6-CSB) -> Net-(BottomStrip1-CS1)
- U1 pad 1: Net-(U1-VDDIO) -> Net-(BottomStrip1-VDDIO)
- U1 pad 10: Net-(U1-VDD) -> Net-(BottomStrip1-VDD)
- U1 pad 2: Net-(U1-SCK) -> Net-(BottomStrip1-SCK1)
- U1 pad 3: Net-(master_connector_input1-GND) -> GND
- U1 pad 4: Net-(U1-SDI) -> Net-(BottomStrip1-MOSI1)
- U1 pad 5: Net-(U1-SDO) -> Net-(BottomStrip1-MISO1)
- U1 pad 6: Net-(U1-CSB) -> Net-(BottomStrip1-CS6)
- U1 pad 8: Net-(master_connector_input1-GND) -> GND
- U1 pad 9: Net-(master_connector_input1-GND) -> GND
- U2 pad 1: Net-(U1-VDDIO) -> Net-(BottomStrip1-VDDIO)
- U2 pad 10: Net-(U1-VDD) -> Net-(BottomStrip1-VDD)
- U2 pad 2: Net-(U1-SCK) -> Net-(BottomStrip1-SCK1)
- U2 pad 3: Net-(master_connector_input1-GND) -> GND
- U2 pad 4: Net-(U1-SDI) -> Net-(BottomStrip1-MOSI1)
- U2 pad 5: Net-(U1-SDO) -> Net-(BottomStrip1-MISO1)
- U2 pad 6: Net-(U2-CSB) -> Net-(BottomStrip1-CS5)
- U2 pad 8: Net-(master_connector_input1-GND) -> GND
- U2 pad 9: Net-(master_connector_input1-GND) -> GND
- U3 pad 1: Net-(U1-VDDIO) -> Net-(BottomStrip1-VDDIO)
- U3 pad 10: Net-(U1-VDD) -> Net-(BottomStrip1-VDD)
- U3 pad 2: Net-(U1-SCK) -> Net-(BottomStrip1-SCK1)
- U3 pad 3: Net-(master_connector_input1-GND) -> GND
- U3 pad 4: Net-(U1-SDI) -> Net-(BottomStrip1-MOSI1)
- U3 pad 5: Net-(U1-SDO) -> Net-(BottomStrip1-MISO1)
- U3 pad 6: Net-(U3-CSB) -> Net-(BottomStrip1-CS4)
- U3 pad 8: Net-(master_connector_input1-GND) -> GND
- U3 pad 9: Net-(master_connector_input1-GND) -> GND
- U4 pad 1: Net-(U1-VDDIO) -> Net-(BottomStrip1-VDDIO)
- U4 pad 10: Net-(U1-VDD) -> Net-(BottomStrip1-VDD)
- U4 pad 2: Net-(U1-SCK) -> Net-(BottomStrip1-SCK1)
- U4 pad 3: Net-(master_connector_input1-GND) -> GND
- U4 pad 4: Net-(U1-SDI) -> Net-(BottomStrip1-MOSI1)
- U4 pad 5: Net-(U1-SDO) -> Net-(BottomStrip1-MISO1)
- U4 pad 6: Net-(U4-CSB) -> Net-(BottomStrip1-CS3)
- U4 pad 8: Net-(master_connector_input1-GND) -> GND
- U4 pad 9: Net-(master_connector_input1-GND) -> GND
- U5 pad 1: Net-(U1-VDDIO) -> Net-(BottomStrip1-VDDIO)
- U5 pad 10: Net-(U1-VDD) -> Net-(BottomStrip1-VDD)
- U5 pad 2: Net-(U1-SCK) -> Net-(BottomStrip1-SCK1)
- U5 pad 3: Net-(master_connector_input1-GND) -> GND
- U5 pad 4: Net-(U1-SDI) -> Net-(BottomStrip1-MOSI1)
- U5 pad 5: Net-(U1-SDO) -> Net-(BottomStrip1-MISO1)
- U5 pad 6: Net-(U5-CSB) -> Net-(BottomStrip1-CS2)
- U5 pad 8: Net-(master_connector_input1-GND) -> GND
- U5 pad 9: Net-(master_connector_input1-GND) -> GND
- U6 pad 1: Net-(U1-VDDIO) -> Net-(BottomStrip1-VDDIO)
- U6 pad 10: Net-(U1-VDD) -> Net-(BottomStrip1-VDD)
- U6 pad 2: Net-(U1-SCK) -> Net-(BottomStrip1-SCK1)
- U6 pad 3: Net-(master_connector_input1-GND) -> GND
- U6 pad 4: Net-(U1-SDI) -> Net-(BottomStrip1-MOSI1)
- U6 pad 5: Net-(U1-SDO) -> Net-(BottomStrip1-MISO1)
- U6 pad 6: Net-(U6-CSB) -> Net-(BottomStrip1-CS1)
- U6 pad 8: Net-(master_connector_input1-GND) -> GND
- U6 pad 9: Net-(master_connector_input1-GND) -> GND
Routing:
- net Net-(BottomStrip1-VDD): track 0.00 -> 378.3 mm, vias 0 -> 12
- net Net-(BottomStrip1-VDDIO): track 0.00 -> 370.4 mm, vias 0 -> 12
- net Net-(BottomStrip1-MOSI1): track 0.00 -> 344.8 mm
- net Net-(BottomStrip1-SCK1): track 0.00 -> 316.4 mm, vias 0 -> 12
- net Net-(BottomStrip1-MISO1): track 0.00 -> 299.4 mm, vias 0 -> 10
- net Net-(BottomStrip1-CS6): track 0.00 -> 289.2 mm
- net Net-(BottomStrip1-CS5): track 0.00 -> 263.4 mm, vias 0 -> 2
- net Net-(BottomStrip1-CS4): track 0.00 -> 232.6 mm, vias 0 -> 2
- net Net-(BottomStrip1-CS3): track 0.00 -> 114.2 mm, vias 0 -> 2
- net Net-(BottomStrip1-CS2): track 0.00 -> 82.4 mm, vias 0 -> 2
- net Net-(BottomStrip1-CS1): track 0.00 -> 51.0 mm, vias 0 -> 2
- net GND: track 0.00 -> 25.0 mm, vias 0 -> 14
- added copper zone on B.Cu, net GND
Other:
- board outline added: 289.3 x 25 mm
- board text added: "Bottom Sensor Strip"
