File: BMP581_PCB/SensorStrip_Bottom/SensorStrip_Bottom.kicad_sch (KiCad schematic)
At the start: 15 parts

Commit message: update strips
Parts:
- BottomStrip1: renamed from master_connector_input1; footprint Connector_PinHeader_1.00mm:PinHeader_1x15_P1.00mm_Vertical_SMD_Pin1Left -> BMP581:Strip_pins_bottom
- R1: renamed from R7; footprint Resistor_SMD:R_01005_0402Metric_Pad0.57x0.30mm_HandSolder -> Resistor_SMD:R_0402_1005Metric
- R2: renamed from R6; footprint Resistor_SMD:R_01005_0402Metric_Pad0.57x0.30mm_HandSolder -> Resistor_SMD:R_0402_1005Metric
- R3: renamed from R5; footprint Resistor_SMD:R_01005_0402Metric_Pad0.57x0.30mm_HandSolder -> Resistor_SMD:R_0402_1005Metric
- R4: footprint Resistor_SMD:R_01005_0402Metric_Pad0.57x0.30mm_HandSolder -> Resistor_SMD:R_0402_1005Metric
- R5: renamed from R3; footprint Resistor_SMD:R_01005_0402Metric_Pad0.57x0.30mm_HandSolder -> Resistor_SMD:R_0402_1005Metric
- R6: renamed from R2; footprint Resistor_SMD:R_01005_0402Metric_Pad0.57x0.30mm_HandSolder -> Resistor_SMD:R_0402_1005Metric
Connections:
- net GND: now also BottomStrip1.2 (GND), U1.3 (GND), U1.8 (GND), U1.9 (GND), U2.3 (GND), U2.8 (GND), U2.9 (GND), U3.3 (GND), U3.8 (GND), U3.9 (GND), U4.3 (GND), U4.8 (GND), U4.9 (GND), U5.3 (GND), U5.8 (GND), U5.9 (GND), U6.3 (GND), U6.8 (GND), U6.9 (GND)
Changed lines of the file:
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@@
     (stroke (width 0) (type default))
   )
+  (global_label "GND" (shape input) (at 415.29 154.94 0) (fields_autoplaced)
+    (effects (font (size 1.27 1.27)) (justify left))
+    (property "Intersheetrefs" "${INTERSHEET_REFS}" (at 422.0663 154.94 0)
+      (effects (font (size 1.27 1.27)) (justify left) hide)
+    )
+  )
   (symbol (lib_id "BMP581_symbol:BMP581") (at 236.22 172.72 0) (unit 1)
     (in_bom yes) (on_board yes) (dnp no) (fields_autoplaced)
@@
   (symbol (lib_id "Device:R") (at 99.06 172.72 0) (unit 1)
     (in_bom yes) (on_board yes) (dnp no) (fields_autoplaced)
-    (property "Reference" "R7" (at 101.6 172.085 0)
+    (property "Reference" "R1" (at 101.6 172.085 0)
       (effects (font (size 1.27 1.27)) (justify left))
     )
@@
       (effects (font (size 1.27 1.27)) (justify left))
     )
-    (property "Footprint" "Resistor_SMD:R_01005_0402Metric_Pad0.57x0.30mm_HandSolder" (at 97.282 172.72 90)
-      (effects (font (size 1.27 1.27)) hide)
-    )
-    (property "Datasheet" "~" (at 99.06 172.72 0)
-      (effects (font (size 1.27 1.27)) hide)
-    )
-    (pin "1")
-    (pin "2")
-    (instances
-      (project "SensorStrip_Bottom"
-        (path "/9da6c076-b28a-4569-841f-5d8b7e795c8c"
-          (reference "R7") (unit 1)
+    (property "Footprint" "Resistor_SMD:R_0402_1005Metric" (at 97.282 172.72 90)
+      (effects (font (size 1.27 1.27)) hide)
+    )
+    (property "Datasheet" "https://www.farnell.com/datasheets/3795017.pdf" (at 99.06 172.72 0)
+      (effects (font (size 1.27 1.27)) hide)
+    )
+    (pin "1")
+    (pin "2")
+    (instances
+      (project "SensorStrip_Bottom"
+        (path "/9da6c076-b28a-4569-841f-5d8b7e795c8c"
+          (reference "R1") (unit 1)
         )
       )
@@
   (symbol (lib_id "BMP581_symbol:std_master_output") (at 458.47 173.99 0) (mirror y) (unit 1)
     (in_bom yes) (on_board yes) (dnp no) (fields_autoplaced)
-    (property "Reference" "master_connector_input1" (at 464.82 170.815 0)
+    (property "Reference" "BottomStrip1" (at 464.82 170.18 0)
       (effects (font (size 1.27 1.27)) (justify right))
     )
-    (property "Value" "std_master_output" (at 464.82 173.355 0)
+    (property "Value" "std_master_output" (at 464.82 172.72 0)
       (effects (font (size 1.27 1.27)) (justify right))
     )
-    (property "Footprint" "Connector_PinHeader_1.00mm:PinHeader_1x15_P1.00mm_Vertical_SMD_Pin1Left" (at 458.47 173.99 0)
+    (property "Footprint" "BMP581:Strip_pins_bottom" (at 458.47 173.99 0)
       (effects (font (size 1.27 1.27)) hide)
     )
@@
       (effects (font (size 1.27 1.27)) hide)
     )
-    (pin "3")
-    (pin "1")
+    (pin "1")
+    (pin "10")
     (pin "11")
     (pin "12")
@@
     (pin "15")
     (pin "2")
-    (pin "4")
-    (pin "5")
-    (pin "6")
-    (pin "7")
-    (pin "8")
-    (pin "9")
-    (pin "10")
-    (instances
-      (project "SensorStrip_Bottom"
-        (path "/9da6c076-b28a-4569-841f-5d8b7e795c8c"
-          (reference "master_connector_input1") (unit 1)
+    (pin "3")
+    (pin "4")
+    (pin "5")
+    (pin "6")
+    (pin "7")
+    (pin "8")
+    (pin "9")
+    (instances
+      (project "SensorStrip_Bottom"
+        (path "/9da6c076-b28a-4569-841f-5d8b7e795c8c"
+          (reference "BottomStrip1") (unit 1)
         )
       )
@@
   (symbol (lib_id "Device:R") (at 369.57 172.72 0) (unit 1)
     (in_bom yes) (on_board yes) (dnp no) (fields_autoplaced)
-    (property "Reference" "R2" (at 372.11 172.085 0)
+    (property "Reference" "R6" (at 372.11 172.085 0)
       (effects (font (size 1.27 1.27)) (justify left))
     )
@@
       (effects (font (size 1.27 1.27)) (justify left))
     )
-    (property "Footprint" "Resistor_SMD:R_01005_0402Metric_Pad0.57x0.30mm_HandSolder" (at 367.792 172.72 90)
-      (effects (font (size 1.27 1.27)) hide)
-    )
-    (property "Datasheet" "~" (at 369.57 172.72 0)
-      (effects (font (size 1.27 1.27)) hide)
-    )
-    (pin "1")
-    (pin "2")
-    (instances
-      (project "SensorStrip_Bottom"
-        (path "/9da6c076-b28a-4569-841f-5d8b7e795c8c"
-          (reference "R2") (unit 1)
+    (property "Footprint" "Resistor_SMD:R_0402_1005Metric" (at 367.792 172.72 90)
+      (effects (font (size 1.27 1.27)) hide)
+    )
+    (property "Datasheet" "https://www.farnell.com/datasheets/3795017.pdf" (at 369.57 172.72 0)
+      (effects (font (size 1.27 1.27)) hide)
+    )
+    (pin "1")
+    (pin "2")
+    (instances
+      (project "SensorStrip_Bottom"
+        (path "/9da6c076-b28a-4569-841f-5d8b7e795c8c"
+          (reference "R6") (unit 1)
         )
       )
@@
   (symbol (lib_id "Device:R") (at 308.61 172.72 0) (unit 1)
     (in_bom yes) (on_board yes) (dnp no) (fields_autoplaced)
-    (property "Reference" "R3" (at 311.15 172.085 0)
+    (property "Reference" "R5" (at 311.15 172.085 0)
       (effects (font (size 1.27 1.27)) (justify left))
     )
@@
       (effects (font (size 1.27 1.27)) (justify left))
     )
-    (property "Footprint" "Resistor_SMD:R_01005_0402Metric_Pad0.57x0.30mm_HandSolder" (at 306.832 172.72 90)
-      (effects (font (size 1.27 1.27)) hide)
-    )
-    (property "Datasheet" "~" (at 308.61 172.72 0)
-      (effects (font (size 1.27 1.27)) hide)
-    )
-    (pin "1")
-    (pin "2")
-    (instances
-      (project "SensorStrip_Bottom"
-        (path "/9da6c076-b28a-4569-841f-5d8b7e795c8c"
-          (reference "R3") (unit 1)
+    (property "Footprint" "Resistor_SMD:R_0402_1005Metric" (at 306.832 172.72 90)
+      (effects (font (size 1.27 1.27)) hide)
+    )
+    (property "Datasheet" "https://www.farnell.com/datasheets/3795017.pdf" (at 308.61 172.72 0)
+      (effects (font (size 1.27 1.27)) hide)
+    )
+    (pin "1")
+    (pin "2")
+    (instances
+      (project "SensorStrip_Bottom"
+        (path "/9da6c076-b28a-4569-841f-5d8b7e795c8c"
+          (reference "R5") (unit 1)
         )
       )
@@
   (symbol (lib_id "Device:R") (at 203.2 172.72 0) (unit 1)
     (in_bom yes) (on_board yes) (dnp no) (fields_autoplaced)
-    (property "Reference" "R5" (at 205.74 172.085 0)
+    (property "Reference" "R3" (at 205.74 172.085 0)
       (effects (font (size 1.27 1.27)) (justify left))
     )
@@
       (effects (font (size 1.27 1.27)) (justify left))
     )
-    (property "Footprint" "Resistor_SMD:R_01005_0402Metric_Pad0.57x0.30mm_HandSolder" (at 201.422 172.72 90)
-      (effects (font (size 1.27 1.27)) hide)
-    )
-    (property "Datasheet" "~" (at 203.2 172.72 0)
-      (effects (font (size 1.27 1.27)) hide)
-    )
-    (pin "1")
-    (pin "2")
-    (instances
-      (project "SensorStrip_Bottom"
-        (path "/9da6c076-b28a-4569-841f-5d8b7e795c8c"
-          (reference "R5") (unit 1)
+    (property "Footprint" "Resistor_SMD:R_0402_1005Metric" (at 201.422 172.72 90)
+      (effects (font (size 1.27 1.27)) hide)
+    )
+    (property "Datasheet" "https://www.farnell.com/datasheets/3795017.pdf" (at 203.2 172.72 0)
+      (effects (font (size 1.27 1.27)) hide)
+    )
+    (pin "1")
+    (pin "2")
+    (instances
+      (project "SensorStrip_Bottom"
+        (path "/9da6c076-b28a-4569-841f-5d8b7e795c8c"
+          (reference "R3") (unit 1)
         )
       )
@@
   (symbol (lib_id "Device:R") (at 151.13 172.72 0) (unit 1)
     (in_bom yes) (on_board yes) (dnp no) (fields_autoplaced)
-    (property "Reference" "R6" (at 153.67 172.085 0)
+    (property "Reference" "R2" (at 153.67 172.085 0)
       (effects (font (size 1.27 1.27)) (justify left))
     )
@@
       (effects (font (size 1.27 1.27)) (justify left))
     )
-    (property "Footprint" "Resistor_SMD:R_01005_0402Metric_Pad0.57x0.30mm_HandSolder" (at 149.352 172.72 90)
-      (effects (font (size 1.27 1.27)) hide)
-    )
-    (property "Datasheet" "~" (at 151.13 172.72 0)
-      (effects (font (size 1.27 1.27)) hide)
-    )
-    (pin "1")
-    (pin "2")
-    (instances
-      (project "SensorStrip_Bottom"
-        (path "/9da6c076-b28a-4569-841f-5d8b7e795c8c"
-          (reference "R6") (unit 1)
+    (property "Footprint" "Resistor_SMD:R_0402_1005Metric" (at 149.352 172.72 90)
+      (effects (font (size 1.27 1.27)) hide)
+    )
+    (property "Datasheet" "https://www.farnell.com/datasheets/3795017.pdf" (at 151.13 172.72 0)
+      (effects (font (size 1.27 1.27)) hide)
+    )
+    (pin "1")
+    (pin "2")
+    (instances
+      (project "SensorStrip_Bottom"
+        (path "/9da6c076-b28a-4569-841f-5d8b7e795c8c"
+          (reference "R2") (unit 1)
         )
       )
@@
       (effects (font (size 1.27 1.27)) (justify left))
     )
-    (property "Footprint" "Resistor_SMD:R_01005_0402Metric_Pad0.57x0.30mm_HandSolder" (at 254.762 172.72 90)
-      (effects (font (size 1.27 1.27)) hide)
-    )
-    (property "Datasheet" "~" (at 256.54 172.72 0)
-      (effects (font (size 1.27 1.27)) hide)
-    )
+    (property "Footprint" "Resistor_SMD:R_0402_1005Metric" (at 254.762 172.72 90)
+      (effects (font (size 1.27 1.27)) hide)
+    )
+    (property "Datasheet" "https://www.farnell.com/datasheets/3795017.pdf" (at 256.54 172.72 0)
+      (effects (font (size 1.27 1.27)) hide)
+    )
