File: BMP581_PCB/SensorStrip_Top/SensorStrip_Top.kicad_pcb (KiCad board)
At the start: 2 copper layers, 289.3 x 25 mm, 15 parts

Commit message: Top sensor strip completed v1
Parts:
- removed R1, R2, R3, R4, R5, R6: 10000, Resistor_SMD:R_0402_1005Metric
- added C3: 470nF, Capacitor_SMD:C_0603_1608Metric, F.Cu at (34.2, 111.0)
- added C4: 470nF, Capacitor_SMD:C_0603_1608Metric, F.Cu at (34.2, 113.0)
- added TCS1: TestPoint_Probe, TestPoint:TestPoint_Pad_1.0x1.0mm, F.Cu at (247.8, 117.0)
- added TCS2: TestPoint_Probe, TestPoint:TestPoint_Pad_1.0x1.0mm, F.Cu at (217.2, 118.2)
- added TCS3: TestPoint_Probe, TestPoint:TestPoint_Pad_1.0x1.0mm, F.Cu at (196.5, 118.2)
- added TCS4: TestPoint_Probe, TestPoint:TestPoint_Pad_1.0x1.0mm, F.Cu at (69.0, 119.8)
- added TCS5: TestPoint_Probe, TestPoint:TestPoint_Pad_1.0x1.0mm, F.Cu at (39.8, 121.0)
- added TCS6: TestPoint_Probe, TestPoint:TestPoint_Pad_1.0x1.0mm, F.Cu at (23.2, 124.0)
- added TGND1: TestPoint_Probe, TestPoint:TestPoint_Pad_1.0x1.0mm, F.Cu at (12.2, 131.2)
- added TMISO1: TestPoint_Probe, TestPoint:TestPoint_Pad_1.0x1.0mm, F.Cu at (73.0, 129.8)
- added TMISO2: TestPoint_Probe, TestPoint:TestPoint_Pad_1.0x1.0mm, F.Cu at (98.0, 108.2)
- added TMOSI1: TestPoint_Probe, TestPoint:TestPoint_Pad_1.0x1.0mm, F.Cu at (78.6, 129.8)
- added TMOSI2: TestPoint_Probe, TestPoint:TestPoint_Pad_1.0x1.0mm, F.Cu at (94.5, 108.2)
- added TSCK1: TestPoint_Probe, TestPoint:TestPoint_Pad_1.0x1.0mm, F.Cu at (67.2, 129.8)
- added TSCK2: TestPoint_Probe, TestPoint:TestPoint_Pad_1.0x1.0mm, F.Cu at (101.5, 108.2)
- added TVDD1: TestPoint_Probe, TestPoint:TestPoint_Pad_1.0x1.0mm, F.Cu at (25.8, 109.8)
- added TVDDIO1: TestPoint_Probe, TestPoint:TestPoint_Pad_1.0x1.0mm, F.Cu at (33.5, 108.5)
- added U10: ~, BMP581:BMP581_Landing_Pattern, F.Cu at (206.1, 130.9)
- added U11: ~, BMP581:BMP581_Landing_Pattern, F.Cu at (235.8, 130.9)
- added U12: ~, BMP581:BMP581_Landing_Pattern, F.Cu at (265.4, 130.9)
- added U7: ~, BMP581:BMP581_Landing_Pattern, F.Cu at (28.4, 130.9)
- added U8: ~, BMP581:BMP581_Landing_Pattern, F.Cu at (58.0, 130.9)
- added U9: ~, BMP581:BMP581_Landing_Pattern, F.Cu at (87.7, 130.9)
- moved C1 32.5 mm to (240.0, 111.5), turned to 180 degrees
- moved C2 27.5 mm to (240.0, 109.0), turned to 180 degrees
- moved TopConnector1 14.2 mm to (275.8, 119.0), turned to 25 degrees
Connections:
- net Net-(TopConnector1-CS1) renamed CS1
- net Net-(TopConnector1-CS2) renamed CS2
- net Net-(TopConnector1-CS3) renamed CS3
- net Net-(TopConnector1-CS4) renamed CS4
- net Net-(TopConnector1-CS5) renamed CS5
- net Net-(TopConnector1-CS6) renamed CS6
- net Net-(TopConnector1-MISO) renamed MISO
- net Net-(TopConnector1-MOSI) renamed MOSI
- net Net-(TopConnector1-SCK) renamed SCK
- net Net-(TopConnector1-VDD) renamed VDD
- net Net-(TopConnector1-VDDIO) renamed VDDIO
- TopConnector1 pad 7: unconnected-(TopConnector1-SCK1-Pad7) -> SCK1
- TopConnector1 pad 8: unconnected-(TopConnector1-MISO1-Pad8) -> MISO1
- TopConnector1 pad 9: unconnected-(TopConnector1-MOSI1-Pad9) -> MOSI1
Routing:
- net MISO1: track 0.00 -> 341.3 mm, vias 0 -> 14
- net MOSI1: track 0.00 -> 337.9 mm, vias 0 -> 2
- net SCK1: track 0.00 -> 327.8 mm, vias 0 -> 16
- net MISO: track 402.3 -> 311.4 mm
- net VDD: track 328.6 -> 419.3 mm, vias 10 -> 12
- net VDDIO: track 354.1 -> 440.6 mm, vias 12 -> 34
- net MOSI: track 351.0 -> 322.2 mm, vias 2 -> 14
- net SCK: track 331.3 -> 305.0 mm, vias 10 -> 0
- net CS5: track 258.5 -> 278.4 mm, vias 2 -> 4
- net GND: track 26.5 -> 45.6 mm, vias 14 -> 28
- net CS4: track 229.0 -> 247.3 mm, vias 2 -> 4
- net CS6: track 285.5 -> 303.2 mm, vias 0 -> 2
- net CS2: track 84.0 -> 89.5 mm, vias 2 -> 4
- net CS1: track 54.1 -> 58.2 mm, vias 2 -> 4
- net CS3: vias 2 -> 4
Other:
- board size 289.3 x 25 mm -> 275.8 x 29.5 mm
