File: Experiment_PCB/SensorStrip_Top/SensorStrip_Top.kicad_sch (KiCad schematic)
At the start: 32 parts

Commit message: Incorporate feedback
Parts:
- removed C1: 470nF, Capacitor_SMD:C_0603_1608Metric, symbol Device:C
- removed TVDDIO1: TestPoint_Probe, TestPoint:TestPoint_Pad_1.0x1.0mm, symbol Connector:TestPoint_Probe
- removed TopConnector1: std_master_output, BMP581:Strip_pins_top, symbol BMP581_symbol:std_master_output
- added C10, C11, C12, C13, C14, C15, C16, C17, C18, C19, C2, C20, C21, C22, C23, C24, C25, C5, C6, C7, C8, C9: 100nF, Capacitor_SMD:C_0201_0603Metric, symbol Device:C
- added master_connector_input1: std_master_output, BMP581:Strip_pins_top, symbol BMP581_symbol:std_master_output
- C1: renamed from C2; value 470nF -> 1uF
- C3, C4: value 470nF -> 100nF; footprint Capacitor_SMD:C_0603_1608Metric -> Capacitor_SMD:C_0201_0603Metric
Connections:
- net VDDIO is gone; now on net VDD: C3.2, U1.1 (VDDIO), U10.1 (VDDIO), U11.1 (VDDIO), U12.1 (VDDIO), U2.1 (VDDIO), U3.1 (VDDIO), U4.1 (VDDIO), U5.1 (VDDIO), U6.1 (VDDIO), U7.1 (VDDIO), U8.1 (VDDIO), U9.1 (VDDIO)
- net CS1: now also master_connector_input1.9 (CS1)
- net CS2: now also master_connector_input1.10 (CS2)
- net CS3: now also master_connector_input1.11 (CS3)
- net CS4: now also master_connector_input1.12 (CS4)
- net CS5: now also master_connector_input1.13 (CS5)
- net CS6: now also master_connector_input1.14 (CS6)
- net GND: now also U1.7 (INT), U10.7 (INT), U11.7 (INT), U12.7 (INT), U2.7 (INT), U3.7 (INT), U4.7 (INT), U5.7 (INT), U6.7 (INT), U7.7 (INT), U8.7 (INT), U9.7 (INT), C10.1, C11.1, C12.1, C13.1, C14.1, C15.1, C16.1, C17.1, C18.1, C19.1, C2.1, C20.1, C21.1, C22.1, C23.1, C24.1, C25.1, C5.1, C6.1, C7.1, C8.1, C9.1, master_connector_input1.2 (GND)
- net MISO: now also master_connector_input1.4 (MISO)
- net MISO1: now also master_connector_input1.7 (MISO1)
- net MOSI: now also master_connector_input1.5 (MOSI)
- net MOSI1: now also master_connector_input1.8 (MOSI1)
- net SCK: now also master_connector_input1.3 (SCK)
- net SCK1: now also master_connector_input1.6 (SCK1)
- net VDD: now also C10.2, C11.2, C12.2, C13.2, C14.2, C15.2, C16.2, C17.2, C18.2, C19.2, C2.2, C20.2, C21.2, C22.2, C23.2, C24.2, C25.2, C5.2, C6.2, C7.2, C8.2, C9.2, master_connector_input1.1 (VDD)
Other:
- moved on the sheet: C1
