File: Experiment_PCB/SensorStrip_Top/SensorStrip_Top.kicad_pcb (KiCad board)
At the start: 2 copper layers, 275.8 x 29.5 mm, 32 parts

Commit message: Incorporate feedback
Parts:
- removed TVDDIO1: TestPoint_Probe, TestPoint:TestPoint_Pad_1.0x1.0mm
- removed TopConnector1: std_master_output, BMP581:Strip_pins_top
- added C10: 100nF, Capacitor_SMD:C_0201_0603Metric, F.Cu at (195.8, 108.5)
- added C11: 100nF, Capacitor_SMD:C_0201_0603Metric, F.Cu at (192.5, 107.0)
- added C12: 100nF, Capacitor_SMD:C_0201_0603Metric, F.Cu at (205.5, 128.4)
- added C13: 100nF, Capacitor_SMD:C_0201_0603Metric, F.Cu at (208.4, 129.7)
- added C14: 100nF, Capacitor_SMD:C_0201_0603Metric, F.Cu at (77.3, 108.5)
- added C15: 100nF, Capacitor_SMD:C_0201_0603Metric, F.Cu at (74.2, 106.8)
- added C16: 100nF, Capacitor_SMD:C_0201_0603Metric, F.Cu at (44.5, 107.0)
- added C17: 100nF, Capacitor_SMD:C_0201_0603Metric, F.Cu at (47.8, 108.5)
- added C18: 100nF, Capacitor_SMD:C_0201_0603Metric, F.Cu at (18.2, 108.8)
- added C19: 100nF, Capacitor_SMD:C_0201_0603Metric, F.Cu at (16.8, 106.5)
- added C20: 100nF, Capacitor_SMD:C_0201_0603Metric, F.Cu at (27.9, 128.2)
- added C21: 100nF, Capacitor_SMD:C_0201_0603Metric, F.Cu at (30.8, 129.5)
- added C22: 100nF, Capacitor_SMD:C_0201_0603Metric, F.Cu at (57.3, 127.8)
- added C23: 100nF, Capacitor_SMD:C_0201_0603Metric, F.Cu at (60.4, 129.7)
- added C24: 100nF, Capacitor_SMD:C_0201_0603Metric, F.Cu at (86.9, 127.8)
- added C25: 100nF, Capacitor_SMD:C_0201_0603Metric, F.Cu at (90.0, 129.5)
- added C5: 100nF, Capacitor_SMD:C_0201_0603Metric, F.Cu at (225.8, 108.5)
- added C6: 100nF, Capacitor_SMD:C_0201_0603Metric, F.Cu at (267.8, 129.0)
- added C7: 100nF, Capacitor_SMD:C_0201_0603Metric, F.Cu at (264.7, 128.2)
- added C8: 100nF, Capacitor_SMD:C_0201_0603Metric, F.Cu at (238.1, 129.4)
- added C9: 100nF, Capacitor_SMD:C_0201_0603Metric, F.Cu at (235.1, 128.2)
- added master_connector_input1: std_master_output, BMP581:Strip_pins_top, F.Cu at (277.0, 120.5)
- C1: value 470nF -> 1uF
- C2, C3, C4: value 470nF -> 100nF; footprint Capacitor_SMD:C_0603_1608Metric -> Capacitor_SMD:C_0201_0603Metric
- moved C3 223.9 mm to (254.9, 108.5)
- moved C4 195.0 mm to (222.4, 107.0)
- moved C1 143.5 mm to (95.0, 107.8), turned to 90 degrees
- moved C2 17.3 mm to (252.1, 107.0)
Connections:
- C1 pad 2: VDDIO -> VDD
- C3 pad 2: VDDIO -> VDD
- U1 pad 1: VDDIO -> VDD
- U1 pad 7: unconnected-(U1-INT-Pad7) -> GND
- U10 pad 1: VDDIO -> VDD
- U10 pad 7: unconnected-(U10-INT-Pad7) -> GND
- U11 pad 1: VDDIO -> VDD
- U11 pad 7: unconnected-(U11-INT-Pad7) -> GND
- U12 pad 1: VDDIO -> VDD
- U12 pad 7: unconnected-(U12-INT-Pad7) -> GND
- U2 pad 1: VDDIO -> VDD
- U2 pad 7: unconnected-(U2-INT-Pad7) -> GND
- U3 pad 1: VDDIO -> VDD
- U3 pad 7: unconnected-(U3-INT-Pad7) -> GND
- U4 pad 1: VDDIO -> VDD
- U4 pad 7: unconnected-(U4-INT-Pad7) -> GND
- U5 pad 1: VDDIO -> VDD
- U5 pad 7: unconnected-(U5-INT-Pad7) -> GND
- U6 pad 1: VDDIO -> VDD
- U6 pad 7: unconnected-(U6-INT-Pad7) -> GND
- U7 pad 1: VDDIO -> VDD
- U7 pad 7: unconnected-(U7-INT-Pad7) -> GND
- U8 pad 1: VDDIO -> VDD
- U8 pad 7: unconnected-(U8-INT-Pad7) -> GND
- U9 pad 1: VDDIO -> VDD
- U9 pad 7: unconnected-(U9-INT-Pad7) -> GND
Routing:
- net VDDIO: track 433.0 -> 0.00 mm, vias 34 -> 0
- net VDD: track 409.7 -> 474.3 mm
- net GND: track 43.2 -> 103.0 mm, vias 30 -> 151
- net MOSI1: track 334.9 -> 335.9 mm
- added copper zone on F.Cu, net GND

Commit message: update for file transfer / cleanup some traces
Parts:
- moved C3 0.09 mm to (255.0, 108.5)
Routing:
- net GND: track 103.0 -> 109.7 mm, vias 151 -> 135
- net MISO1: track 337.1 -> 339.8 mm, vias 12 -> 11
- net MOSI1: track 335.9 -> 334.1 mm, vias 2 -> 1
- net MISO: track 303.1 -> 304.7 mm
- net VDD: track 474.3 -> 475.6 mm
- net SCK: track 301.7 -> 302.4 mm
- net CS3: track 114.0 -> 114.6 mm
- net SCK1: vias 14 -> 13

Commit message: transfer files to laptop for order
Parts:
- added REF**: MountingHole_2.2mm_M2_ISO7380, MountingHole:MountingHole_2.2mm_M2_ISO7380, F.Cu at (43.2, 130.5)
- added REF**: MountingHole_2.2mm_M2_ISO7380, MountingHole:MountingHole_2.2mm_M2_ISO7380, F.Cu at (35.0, 110.0)
Routing:
- net GND: vias 135 -> 108

Commit message: Ordered PCBs
Parts:
- added REF**: MountingHole_2.2mm_M2_ISO7380, MountingHole:MountingHole_2.2mm_M2_ISO7380, F.Cu at (242.5, 109.8)
- added REF**: MountingHole_2.2mm_M2_ISO7380, MountingHole:MountingHole_2.2mm_M2_ISO7380, F.Cu at (250.2, 130.2)
