File: Experiment_PCB/SensorStrip_Bottom/SensorStrip_Bottom.kicad_pcb (KiCad board)
At the start: 2 copper layers, 275.8 x 29.5 mm, 32 parts

Commit message: Incorporate feedback
Parts:
- removed BottomStrip1: std_master_output, BMP581:Strip_pins_bottom
- removed VDDIO1: TestPoint_Probe, TestPoint:TestPoint_Pad_1.0x1.0mm
- added C10: 100nF, Capacitor_SMD:C_0201_0603Metric, F.Cu at (178.1, 107.0)
- added C11: 100nF, Capacitor_SMD:C_0201_0603Metric, F.Cu at (175.2, 105.8)
- added C12: 100nF, Capacitor_SMD:C_0201_0603Metric, F.Cu at (191.3, 85.8)
- added C13: 100nF, Capacitor_SMD:C_0201_0603Metric, F.Cu at (188.2, 84.1)
- added C14: 100nF, Capacitor_SMD:C_0201_0603Metric, F.Cu at (27.2, 105.6)
- added C15: 100nF, Capacitor_SMD:C_0201_0603Metric, F.Cu at (30.1, 107.2)
- added C16: 100nF, Capacitor_SMD:C_0201_0603Metric, F.Cu at (59.6, 107.0)
- added C17: 100nF, Capacitor_SMD:C_0201_0603Metric, F.Cu at (56.8, 105.6)
- added C18: 100nF, Capacitor_SMD:C_0201_0603Metric, F.Cu at (72.6, 85.8)
- added C19: 100nF, Capacitor_SMD:C_0201_0603Metric, F.Cu at (69.8, 84.1)
- added C20: 100nF, Capacitor_SMD:C_0201_0603Metric, F.Cu at (40.0, 84.1)
- added C21: 100nF, Capacitor_SMD:C_0201_0603Metric, F.Cu at (43.3, 85.8)
- added C22: 100nF, Capacitor_SMD:C_0201_0603Metric, F.Cu at (13.1, 85.5)
- added C23: 100nF, Capacitor_SMD:C_0201_0603Metric, F.Cu at (10.5, 84.3)
- added C24: 100nF, Capacitor_SMD:C_0201_0603Metric, F.Cu at (-2.50, 105.0)
- added C25: 100nF, Capacitor_SMD:C_0201_0603Metric, F.Cu at (0.75, 107.2)
- added C5: 100nF, Capacitor_SMD:C_0201_0603Metric, F.Cu at (234.5, 105.6)
- added C6: 100nF, Capacitor_SMD:C_0201_0603Metric, F.Cu at (220.6, 85.5)
- added C7: 100nF, Capacitor_SMD:C_0201_0603Metric, F.Cu at (217.8, 84.3)
- added C8: 100nF, Capacitor_SMD:C_0201_0603Metric, F.Cu at (204.8, 105.5)
- added C9: 100nF, Capacitor_SMD:C_0201_0603Metric, F.Cu at (207.8, 107.0)
- added master_connector_input1: std_master_output, BMP581:Strip_pins_bottom, F.Cu at (261.2, 93.5)
- C1: value 470nF -> 1uF
- C2, C3, C4: value 470nF -> 100nF; footprint Capacitor_SMD:C_0603_1608Metric -> Capacitor_SMD:C_0201_0603Metric
- moved C3 238.3 mm to (247.2, 84.6), turned to 90 degrees
- moved C4 223.9 mm to (237.3, 107.0)
- moved C1 152.5 mm to (68.0, 105.0), turned to -90 degrees
- moved C2 37.7 mm to (250.1, 85.5), turned to 180 degrees
Connections:
- C2 pad 2: VDDIO -> VDD
- C3 pad 2: VDDIO -> VDD
- U1 pad 1: VDDIO -> VDD
- U1 pad 7: unconnected-(U1-INT-Pad7) -> GND
- U10 pad 1: VDDIO -> VDD
- U10 pad 7: unconnected-(U10-INT-Pad7) -> GND
- U11 pad 1: VDDIO -> VDD
- U11 pad 7: unconnected-(U11-INT-Pad7) -> GND
- U12 pad 1: VDDIO -> VDD
- U12 pad 7: unconnected-(U12-INT-Pad7) -> GND
- U2 pad 1: VDDIO -> VDD
- U2 pad 7: unconnected-(U2-INT-Pad7) -> GND
- U3 pad 1: VDDIO -> VDD
- U3 pad 7: unconnected-(U3-INT-Pad7) -> GND
- U4 pad 1: VDDIO -> VDD
- U4 pad 7: unconnected-(U4-INT-Pad7) -> GND
- U5 pad 1: VDDIO -> VDD
- U5 pad 7: unconnected-(U5-INT-Pad7) -> GND
- U6 pad 1: VDDIO -> VDD
- U6 pad 7: unconnected-(U6-INT-Pad7) -> GND
- U7 pad 1: VDDIO -> VDD
- U7 pad 7: unconnected-(U7-INT-Pad7) -> GND
- U8 pad 1: VDDIO -> VDD
- U8 pad 7: unconnected-(U8-INT-Pad7) -> GND
- U9 pad 1: VDDIO -> VDD
- U9 pad 7: unconnected-(U9-INT-Pad7) -> GND
Routing:
- net VDDIO: track 436.7 -> 0.00 mm, vias 36 -> 0
- net VDD: track 410.1 -> 478.7 mm
- net GND: track 44.3 -> 110.8 mm, vias 30 -> 196
- net MISO1: track 318.9 -> 320.2 mm
- net MOSI1: track 329.8 -> 330.6 mm
- net CS2: track 80.1 -> 80.7 mm
- net CS3: track 109.2 -> 109.7 mm
- net CS5: track 267.8 -> 268.3 mm
- added copper zone on F.Cu, net GND

Commit message: update for file transfer / cleanup some traces
Parts:
- moved C18 0.31 mm to (72.9, 85.8)
Routing:
- net GND: track 110.8 -> 119.3 mm
- net MISO1: track 320.2 -> 324.6 mm, vias 12 -> 11
- net MOSI1: track 330.6 -> 332.9 mm, vias 2 -> 1
- net SCK1: track 329.4 -> 329.6 mm, vias 12 -> 11

Commit message: transfer files to laptop for order
Parts:
- added REF**: MountingHole_2.2mm_M2_ISO7380, MountingHole:MountingHole_2.2mm_M2_ISO7380, F.Cu at (27.5, 83.5)
- added REF**: MountingHole_2.2mm_M2_ISO7380, MountingHole:MountingHole_2.2mm_M2_ISO7380, F.Cu at (19.2, 104.0)
Routing:
- net GND: track 119.3 -> 119.9 mm, vias 196 -> 118
- net VDD: vias 16 -> 14

Commit message: Ordered PCBs
Parts:
- added REF**: MountingHole_2.2mm_M2_ISO7380, MountingHole:MountingHole_2.2mm_M2_ISO7380, F.Cu at (234.5, 83.8)
- added REF**: MountingHole_2.2mm_M2_ISO7380, MountingHole:MountingHole_2.2mm_M2_ISO7380, F.Cu at (226.8, 104.2)
Routing:
- net GND: vias 118 -> 116
